Commit message: 修改了速度闭环,加了测试代码,目前误差较大问题已解决,主要原因是速度未闭环,通信无异常

File: src/if_arm_lite/urdf/if_arm_lite.urdf (robot description, URDF)
Before this commit: robot if_arm_lite, 7 links, 6 joints
Joints:
- joint joint1: limit lower=-3.141592653589793 upper=2.6179938779914944 effort=100 velocity=1 -> lower=-3.161592653589793 upper=2.637993877991494 effort=100 velocity=1.047197551196598
- joint joint2: limit lower=-2.6179938779914944 upper=0 effort=100 velocity=1 -> lower=-2.637993877991494 upper=0.020000000000000 effort=100 velocity=1.047197551196598
- joint joint3: limit lower=0 upper=3.141592653589793 effort=100 velocity=1 -> lower=-0.020000000000000 upper=3.161592653589793 effort=100 velocity=1.047197551196598
- joint joint4: limit lower=-1.5707963267948966 upper=1.3962634015954636 effort=100 velocity=1 -> lower=-1.590796326794897 upper=1.416263401595464 effort=100 velocity=1.047197551196598
- joint joint5: limit lower=-0.7853981633974483 upper=0.7853981633974483 effort=100 velocity=1 -> lower=-0.805398163397448 upper=0.805398163397448 effort=100 velocity=1.047197551196598
- joint joint6: limit lower=-3.14 upper=3.14 effort=100 velocity=1 -> lower=-3.160000000000000 upper=3.160000000000000 effort=100 velocity=1.047197551196598

File: src/if_arm_lite_moveit_config/config/if_arm_lite.ros2_control.xacro (robot description, xacro)
@@ -5,9 +5,16 @@
         <ros2_control name="${name}" type="system">
             <hardware>
-                <!-- By default, set up controllers for simulation. This won't work on real hardware -->
-                <plugin>mock_components/GenericSystem</plugin>
+                <plugin>if_arm_hardware/IfArmHardware</plugin>
+                <param name="can_interface">can0</param>
+                <param name="motor_ids">1,2,3,4,5,6</param>
+                <param name="gear_ratios">19,23,19,15,15,15</param>
+                <param name="directions">1,1,1,-1,1,1</param>
+                <param name="zero_offsets">0.0250,0.0002,-0.0126,0.0066,-0.1923,6.8574</param>
+                <param name="max_motor_rpm">1000</param>
+                <!-- 电机侧速度斜率，单位 RPM/s（电机轴），X 固件范围 1~65535；取上限 = 基本不额外限制加速度 -->
+                <param name="default_acc">65535</param>
             </hardware>
             <joint name="joint1">
-                <command_interface name="position"/>
+                <command_interface name="velocity"/>
                 <state_interface name="position">
                   <param name="initial_value">${initial_positions['joint1']}</param>
@@ -16,5 +23,5 @@
             </joint>
             <joint name="joint2">
-                <command_interface name="position"/>
+                <command_interface name="velocity"/>
                 <state_interface name="position">
                   <param name="initial_value">${initial_positions['joint2']}</param>
@@ -23,5 +30,5 @@
             </joint>
             <joint name="joint3">
-                <command_interface name="position"/>
+                <command_interface name="velocity"/>
                 <state_interface name="position">
                   <param name="initial_value">${initial_positions['joint3']}</param>
@@ -30,5 +37,5 @@
             </joint>
             <joint name="joint4">
-                <command_interface name="position"/>
+                <command_interface name="velocity"/>
                 <state_interface name="position">
                   <param name="initial_value">${initial_positions['joint4']}</param>
@@ -37,5 +44,5 @@
             </joint>
             <joint name="joint5">
-                <command_interface name="position"/>
+                <command_interface name="velocity"/>
                 <state_interface name="position">
                   <param name="initial_value">${initial_positions['joint5']}</param>
@@ -44,5 +51,5 @@
             </joint>
             <joint name="joint6">
-                <command_interface name="position"/>
+                <command_interface name="velocity"/>
                 <state_interface name="position">
                   <param name="initial_value">${initial_positions['joint6']}</param>
